File: fmc.kicad_sch (KiCad schematic)
At the start: 22 parts, among them P1 ASP-134488-01, Q1 FDN335N, Q2 FDN335N

Commit message: Changed layout, added 12V and Heart LEDs
Parts:
- added C1: 22uF, Capacitor_SMD:C_0805_2012Metric, symbol Device:C_Small
- added D4, D5: Green, LED_SMD:LED_0603_1608Metric, symbol Device:LED
- added Q3: FDN335N, Package_TO_SOT_SMD:SOT-23, symbol Transistor_FET:Q_NMOS_GSD
- added R1: 1k, Resistor_SMD:R_0603_1608Metric, symbol Device:R_Small_US
- added R2: 8.2k, Resistor_SMD:R_0603_1608Metric, symbol Device:R_Small_US
- added R3, R4, R5: 100k, Resistor_SMD:R_0603_1608Metric, symbol Device:R_Small_US
- D1, D2, D3: value LED_Green -> Green
Connections:
- net GND: now also C1.2, D5.1 (K), Q3.2 (S), R3.1, R4.1, R5.1
- net VDD3P3V: now also R1.2
- net HEARTBEAT: now reaches P1.C27
- net HEARTBEAT: now also Q3.1 (G), R5.2
- net P1_12P0V renamed 12P0V
- net 12P0V: now also R2.2
- net P1_3P3VAUX renamed 3P3VAUX
- net P1_PG_C2M renamed PG_C2M
- net PG_C2M: now also R3.2
- net P1_PRSNT renamed PRSNT
- net P1_TDI renamed TDI
- net P1_TDO renamed TDO
- net P1_VADJ renamed VADJ
- net VADJ: now also C1.1, R4.2
- new net: D4.1 (K), Q3.3 (D)
- new net: D4.2 (A), R1.1
- new net: D5.2 (A), R2.1
Other:
- note added: "Bulk Power"
- note added: "Power/Heartbeat LEDs"
- note removed: "Bulk Power Filtering"
- note removed: "Status"
- moved on the sheet: C34, C35, D1, D2, D3, H1, H2, H3, H4, P1A, P1B, P1C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

Commit message: Add slotted mounting hole footprints for marble alignment
Parts:
- H1: footprint MountingHole:MountingHole_2.7mm_M2.5_Pad -> rf-input-fmc:MountingHole_3.0mm_M2.5_Pad_3.3mm_MarbleSlot
- H2: footprint rf-input-fmc:MountingHole_2.7mm_M2.5_Pad_Marble_Slot -> rf-input-fmc:MountingHole_3.0mm_M2.5_Pad_3.3mm_MarbleSlot
- H3, H4: footprint rf-input-fmc:MountingHole_2.7mm_Pad_3.1mm -> rf-input-fmc:MountingHole_3.0mm_3.8mm_Pad_3.3mm_MarbleSlot
Changed lines of the file:
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@@
 			)
 		)
-		(property "Footprint" "rf-input-fmc:MountingHole_2.7mm_Pad_3.1mm"
+		(property "Footprint" "rf-input-fmc:MountingHole_3.0mm_3.8mm_Pad_3.3mm_MarbleSlot"
 			(at 66.04 226.06 0)
 			(effects
@@
 			)
 		)
-		(property "Footprint" "rf-input-fmc:MountingHole_2.7mm_M2.5_Pad_Marble_Slot"
+		(property "Footprint" "rf-input-fmc:MountingHole_3.0mm_M2.5_Pad_3.3mm_MarbleSlot"
 			(at 66.04 213.36 0)
 			(effects
@@
 			)
 		)
-		(property "Footprint" "rf-input-fmc:MountingHole_2.7mm_Pad_3.1mm"
+		(property "Footprint" "rf-input-fmc:MountingHole_3.0mm_3.8mm_Pad_3.3mm_MarbleSlot"
 			(at 66.04 238.76 0)
 			(effects
@@
 			)
 		)
-		(property "Footprint" "MountingHole:MountingHole_2.7mm_M2.5_Pad"
+		(property "Footprint" "rf-input-fmc:MountingHole_3.0mm_M2.5_Pad_3.3mm_MarbleSlot"
 			(at 66.04 200.66 0)
 			(effects
