File: fmc.kicad_sch (KiCad schematic)
At the start: 31 parts, among them P1 ASP-134488-01, Q1 FDN335N, Q2 FDN335N, Q3 FDN335N

Commit message: Changed 22uF to 1210
Parts:
- C1, C34, C35: footprint Capacitor_SMD:C_0805_2012Metric -> Capacitor_SMD:C_1210_3225Metric; MPN GRM21BR61E226ME44L -> MSASG32MSB5226MPNA01; Manufacturer Murata Electronics -> Taiyo Yuden
Changed lines of the file:
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@@
 			)
 		)
-		(property "Footprint" "Capacitor_SMD:C_0805_2012Metric"
+		(property "Footprint" "Capacitor_SMD:C_1210_3225Metric"
 			(at 35.56 210.82 0)
 			(effects
@@
 			)
 		)
-		(property "Description" "CAP CER 22UF 25V X5R 0805"
+		(property "Description" "CAP CER 22UF 35V X5R 1210"
 			(at 35.56 210.82 0)
 			(effects
@@
 			)
 		)
-		(property "MPN" "GRM21BR61E226ME44L"
+		(property "MPN" "MSASG32MSB5226MPNA01"
 			(at 35.56 210.82 0)
 			(effects
@@
 			)
 		)
-		(property "Manufacturer" "Murata Electronics"
+		(property "Manufacturer" "Taiyo Yuden"
 			(at 35.56 210.82 0)
 			(effects
@@
 			)
 		)
-		(property "Footprint" "Capacitor_SMD:C_0805_2012Metric"
+		(property "Footprint" "Capacitor_SMD:C_1210_3225Metric"
 			(at 35.56 236.22 0)
 			(effects
@@
 			)
 		)
-		(property "Description" "CAP CER 22UF 25V X5R 0805"
+		(property "Description" "CAP CER 22UF 35V X5R 1210"
 			(at 35.56 236.22 0)
 			(effects
@@
 			)
 		)
-		(property "MPN" "GRM21BR61E226ME44L"
+		(property "MPN" "MSASG32MSB5226MPNA01"
 			(at 35.56 236.22 0)
 			(effects
@@
 			)
 		)
-		(property "Manufacturer" "Murata Electronics"
+		(property "Manufacturer" "Taiyo Yuden"
 			(at 35.56 236.22 0)
 			(effects
@@
 			)
 		)
-		(property "Footprint" "Capacitor_SMD:C_0805_2012Metric"
+		(property "Footprint" "Capacitor_SMD:C_1210_3225Metric"
 			(at 35.56 184.15 0)
 			(effects
@@
 			)
 		)
-		(property "Description" "CAP CER 22UF 25V X5R 0805"
+		(property "Description" "CAP CER 22UF 35V X5R 1210"
 			(at 35.56 184.15 0)
 			(effects
@@
 			)
 		)
-		(property "MPN" "GRM21BR61E226ME44L"
+		(property "MPN" "MSASG32MSB5226MPNA01"
 			(at 35.56 184.15 0)
 			(effects
@@
 			)
 		)
-		(property "Manufacturer" "Murata Electronics"
+		(property "Manufacturer" "Taiyo Yuden"
 			(at 35.56 184.15 0)
 			(effects
