File: fmc-template.kicad_pcb (KiCad board)
At the start: 6 copper layers, 84 x 69 mm, 31 parts, among them J19 WP Jumper, P1 ASP-134488-01, Q1 FDN335N, Q2 FDN335N, U9 AT24C64D

Commit message: update pcb from sch
Connections:
- P1 pad C30: /FMC/EEPROM_SCL -> /EEPROM/SCL
- P1 pad C31: /FMC/EEPROM_SDA -> /EEPROM/SDA
- P1 pad C34: /FMC/EEPROM_GA0 -> /EEPROM/GA0
- P1 pad D35: /FMC/EEPROM_GA1 -> /EEPROM/GA1
Routing:
- net /FMC/EEPROM_SDA: track 17.6 -> 0.00 mm, vias 1 -> 0
- net /EEPROM/SDA: track 0.00 -> 17.6 mm, vias 0 -> 1
- net /FMC/EEPROM_SCL: track 16.1 -> 0.00 mm, vias 1 -> 0
- net /EEPROM/SCL: track 0.00 -> 16.1 mm, vias 0 -> 1
- net /FMC/EEPROM_GA0: track 8.83 -> 0.00 mm, vias 1 -> 0
- net /EEPROM/GA0: track 0.00 -> 8.83 mm, vias 0 -> 1
- net /FMC/EEPROM_GA1: track 7.88 -> 0.00 mm, vias 1 -> 0
- net /EEPROM/GA1: track 0.00 -> 7.88 mm, vias 0 -> 1
